File: Flow Shims/hardware/controller/controller.kicad_pcb (KiCad board)
At the start: 2 copper layers, 180 x 41 mm, 58 parts, among them J1 Conn_01x02_Pin, J2 Nano-Fit, J22 5.5mm x 2.1mm, J3 Nano-Fit, J4 USB_B, J8 Conn_02x07_Odd_Even, U1 LMV321, U23 LM317_SOT-223, U24 LM337_SOT223, U25 LM317_SOT-223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

Commit message: All boards DRC/ERC clean
Parts:
- added D3: 1N4148W, Diode_SMD:D_SOD-123, F.Cu at (185.2, 36.2)
- added K1: G5NB, Relay_THT:Relay_SPST_Omron_G5NB, F.Cu at (188.0, 33.7)
- added Q1: BSS138, Package_TO_SOT_SMD:SOT-23, F.Cu at (182.0, 37.5)
Connections:
- J1 pad 1: VD -> Net-(J1-Pin_1)
- U3 pad 13: unconnected-(U3-PA7-Pad13) -> /VD_EN
- U3 pad 16: /VTEMP -> unconnected-(U3-PB2-Pad16)
- U3 pad 19: /EN1_0 -> /VTEMP
- U3 pad 20: unconnected-(U3-PA10-Pad20) -> /EN1_0
Routing:
- net /VD_EN: track 0.00 -> 45.1 mm, vias 0 -> 2
- net +15V: track 230.0 -> 242.1 mm, vias 5 -> 6
- net Net-(D3-A): track 0.00 -> 6.42 mm
- net /VTEMP: track 133.9 -> 139.6 mm
- net GND: track 26.3 -> 29.3 mm, vias 50 -> 55
- net /EN1_0: track 127.9 -> 128.8 mm
- added copper zone on F.Cu, net Net-(J1-Pin_1)
Other:
- board text added: "Thermal Shim Controller BioMEMS 2026"
