File: Flow Shims/hardware/controller/controller.kicad_sch (KiCad schematic)
At the start: 25 parts, among them J1 Conn_01x02_Pin, J2 Nano-Fit, J3 Nano-Fit, J4 USB_B, J8 Conn_02x07_Odd_Even, U1 LMV321, U3 STM32L052K8Ux, Y1 Crystal_GND24

Commit message: All boards DRC/ERC clean
Parts:
- added D3: 1N4148W, Diode_SMD:D_SOD-123, symbol Diode:1N4148W
- added K1: G5NB, Relay_THT:Relay_SPST_Omron_G5NB, symbol Relay:G5NB
- added Q1: BSS138, Package_TO_SOT_SMD:SOT-23, symbol Transistor_FET:BSS138
- added R2: 10k, symbol Device:R_Small
Connections:
- net +15V: now also D3.1 (K), K1.A1
- net EN1_0: now also U3.20 (PA10); no longer U3.19 (PA9)
- net GND: now also Q1.2 (S), R2.2
- net VD: now also K1.13; no longer J1.1 (Pin_1)
- net VTEMP: now also U3.19 (PA9); no longer U3.16 (PB2)
- net VD_EN: now reaches U3.13 (PA7)
- net VD_EN: now also Q1.1 (G), R2.1
- new net: J1.1 (Pin_1), K1.14
- new net: D3.2 (A), K1.A2, Q1.3 (D)
- no-connect marks 12 -> 11
