File: Flow Shims/hardware/controller/psu.kicad_sch (KiCad schematic)
At the start: 33 parts, among them J22 5.5mm x 2.1mm, U23 LM317_SOT-223, U24 LM337_SOT223, U25 LM317_SOT-223

Commit message: Add firmware
Parts:
- R71, R72: value 374 -> 2.2k
- R73, R74: value 124 -> 200
- R75: value 374 -> 3.3k
- R76: value 124 -> 2k
Changed lines of the file:
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@@
 			)
 		)
-		(property "Value" "124"
+		(property "Value" "2k"
 			(at 226.822 71.12 0)
 			(show_name no)
@@
 			)
 		)
-		(property "Value" "374"
+		(property "Value" "3.3k"
 			(at 210.566 81.026 0)
 			(show_name no)
@@
 			)
 		)
-		(property "Value" "124"
+		(property "Value" "200"
 			(at 170.942 71.12 0)
 			(show_name no)
@@
 			)
 		)
-		(property "Value" "374"
+		(property "Value" "2.2k"
 			(at 154.686 81.026 0)
 			(show_name no)
@@
 			)
 		)
-		(property "Value" "374"
+		(property "Value" "2.2k"
 			(at 154.432 91.186 0)
 			(show_name no)
@@
 			)
 		)
-		(property "Value" "124"
+		(property "Value" "200"
 			(at 170.688 100.076 0)
 			(show_name no)
