File: Flow Shims/hardware/heater17/element.kicad_sch (KiCad schematic)
At the start: 3 parts, among them Q1 NVTFS5116PL, U3 TSZ181

Commit message: All boards DRC/ERC clean
Changed lines of the file:
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@@
-	(wire
-		(pts
-			(xy 5.1588 2.0957) (xy 7.6988 2.0957)
-		)
-		(stroke
-			(width 0)
-			(type default)
-		)
-	)
 	(wire
 		(pts
@@
 		)
 	)
-	(label "VG10"
-		(at 5.1588 2.0957 180)
-		(effects
-			(font
-				(size 1.27 1.27)
-			)
-			(justify right bottom)
-		)
-	)
