File: Flow Shims/hardware/heater17/heater.kicad_pcb (KiCad board)
At the start: 4 copper layers, 19 x 112.5 mm, 60 parts, among them J1 Conn_01x03, J2 Nano-Fit, Q1 NVTFS5116PL, Q10 NVTFS5116PL, Q11 NVTFS5116PL, Q12 NVTFS5116PL, Q13 NVTFS5116PL, Q14 NVTFS5116PL, Q15 NVTFS5116PL, Q16 NVTFS5116PL, Q17 NVTFS5116PL, Q2 NVTFS5116PL, Q3 NVTFS5116PL, Q4 NVTFS5116PL, Q5 NVTFS5116PL, Q6 NVTFS5116PL, Q7 NVTFS5116PL, Q8 NVTFS5116PL, Q9 NVTFS5116PL, U1 ADG5206, U10 TSZ181, U11 TSZ181, U12 TSZ181, U13 TSZ181, U14 TSZ181, U15 TSZ181, U16 TSZ181, U17 TSZ181, U18 TSZ181, U19 TSZ181, U2 ADG5206, U3 TSZ181, U4 TSZ181, U5 TSZ181, U6 TSZ181, U7 TSZ181, U8 TSZ181, U9 TSZ181

Commit message: All boards DRC/ERC clean
Parts:
- U10, U11, U12, U13, U14, U15, U16, U17, U18, U19, U3, U4, U5, U6, U7, U8, U9: footprint Package_DFN_QFN:DFN-6_1.3x1.2mm_P0.4mm -> thermalshims:DFN-6_1.3x1.2mm_P0.4mm-narrow
Routing:
- net /EN1: track 70.2 -> 59.3 mm, vias 3 -> 1
- net GND: track 90.4 -> 92.2 mm, vias 39 -> 40
- net Net-(U11--): track 7.20 -> 6.69 mm
- net /A0: track 81.7 -> 81.4 mm, vias 4 -> 3
