File: Flow Shims/hardware/heater25/element.kicad_sch (KiCad schematic)
At the start: 3 parts, among them Q1 NVTFS5116PL, U3 TSZ181

Commit message: All boards DRC/ERC clean
Parts:
- U3: footprint Package_DFN_QFN:DFN-6_1.3x1.2mm_P0.4mm -> thermalshims:DFN-6_1.3x1.2mm_P0.4mm-narrow
Changed lines of the file:
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@@
 	(wire
 		(pts
-			(xy 5.1588 2.0957) (xy 7.6988 2.0957)
+			(xy 170.18 86.36) (xy 170.18 87.63)
 		)
 		(stroke
@@
 	(wire
 		(pts
-			(xy 170.18 86.36) (xy 170.18 87.63)
+			(xy 138.43 83.82) (xy 138.43 96.52)
 		)
 		(stroke
@@
 	(wire
 		(pts
-			(xy 138.43 83.82) (xy 138.43 96.52)
+			(xy 162.56 96.52) (xy 162.56 81.28)
 		)
 		(stroke
@@
 	(wire
 		(pts
-			(xy 162.56 96.52) (xy 162.56 81.28)
+			(xy 158.75 81.28) (xy 162.56 81.28)
 		)
 		(stroke
@@
 	(wire
 		(pts
-			(xy 158.75 81.28) (xy 162.56 81.28)
+			(xy 132.08 78.74) (xy 143.51 78.74)
 		)
 		(stroke
@@
 	(wire
 		(pts
-			(xy 132.08 78.74) (xy 143.51 78.74)
+			(xy 132.08 78.74) (xy 132.08 80.01)
 		)
 		(stroke
@@
 	(wire
 		(pts
-			(xy 132.08 78.74) (xy 132.08 80.01)
+			(xy 143.51 83.82) (xy 138.43 83.82)
 		)
 		(stroke
@@
 	(wire
 		(pts
-			(xy 143.51 83.82) (xy 138.43 83.82)
+			(xy 138.43 96.52) (xy 162.56 96.52)
 		)
 		(stroke
@@
 	(wire
 		(pts
-			(xy 138.43 96.52) (xy 162.56 96.52)
+			(xy 123.19 78.74) (xy 132.08 78.74)
 		)
 		(stroke
@@
 	(wire
 		(pts
-			(xy 123.19 78.74) (xy 132.08 78.74)
+			(xy 148.59 71.12) (xy 148.59 73.66)
 		)
 		(stroke
@@
 	(wire
 		(pts
-			(xy 148.59 71.12) (xy 148.59 73.66)
+			(xy 170.18 68.58) (xy 170.18 76.2)
 		)
 		(stroke
@@
 	(wire
 		(pts
-			(xy 170.18 68.58) (xy 170.18 76.2)
+			(xy 132.08 85.09) (xy 132.08 86.36)
 		)
 		(stroke
 			(width 0)
 			(type default)
-		)
-	)
-	(wire
-		(pts
-			(xy 132.08 85.09) (xy 132.08 86.36)
-		)
-		(stroke
-			(width 0)
-			(type default)
-		)
-	)
-	(label "VG10"
-		(at 5.1588 2.0957 180)
-		(effects
-			(font
-				(size 1.27 1.27)
-			)
-			(justify right bottom)
 		)
 	)
@@
 			)
 		)
-		(property "Footprint" "Package_DFN_QFN:DFN-6_1.3x1.2mm_P0.4mm"
+		(property "Footprint" "thermalshims:DFN-6_1.3x1.2mm_P0.4mm-narrow"
 			(at 151.13 81.28 0)
 			(hide yes)
