File: Flow Shims/hardware/heater25/heater.kicad_pcb (KiCad board)
At the start: 4 copper layers, 19 x 112.5 mm, 84 parts, among them J1 Conn_01x03, J2 Nano-Fit, Q1 NVTFS5116PL, Q10 NVTFS5116PL, Q11 NVTFS5116PL, Q12 NVTFS5116PL, Q13 NVTFS5116PL, Q14 NVTFS5116PL, Q15 NVTFS5116PL, Q16 NVTFS5116PL, Q17 NVTFS5116PL, Q18 NVTFS5116PL, Q19 NVTFS5116PL, Q2 NVTFS5116PL, Q20 NVTFS5116PL, Q21 NVTFS5116PL, Q22 NVTFS5116PL, Q23 NVTFS5116PL, Q24 NVTFS5116PL, Q25 NVTFS5116PL, Q3 NVTFS5116PL, Q4 NVTFS5116PL, Q5 NVTFS5116PL, Q6 NVTFS5116PL, Q7 NVTFS5116PL, Q8 NVTFS5116PL, Q9 NVTFS5116PL, U1 ADG5206, U10 TSZ181, U11 TSZ181, U12 TSZ181, U13 TSZ181, U14 TSZ181, U15 TSZ181, U16 TSZ181, U17 TSZ181, U18 TSZ181, U19 TSZ181, U2 ADG5206, U20 TSZ181, U21 TSZ181, U22 TSZ181, U23 TSZ181, U24 TSZ181, U25 TSZ181, U26 TSZ181, U27 TSZ181, U3 TSZ181, U4 TSZ181, U5 TSZ181, U6 TSZ181, U7 TSZ181, U8 TSZ181, U9 TSZ181

Commit message: All boards DRC/ERC clean
Parts:
- U10, U11, U12, U13, U14, U15, U16, U17, U18, U19, U20, U21, U22, U23, U24, U25, U26, U27, U3, U4, U5, U6, U7, U8, U9: footprint thermalshims:DFN-6_1.3x1.2mm_P0.4mm -> thermalshims:DFN-6_1.3x1.2mm_P0.4mm-narrow
Routing:
- net /EN1: track 71.0 -> 60.2 mm, vias 3 -> 1
- net /EN0: track 19.3 -> 18.8 mm
- net VD: vias 85 -> 84
- net /VG5: vias 1 -> 0
