File: Flow Shims/hardware/temp_sensors25/temp_sensors.kicad_pcb (KiCad board)
At the start: 2 copper layers, 6 x 113 mm, 52 parts, among them J1 Conn_01x03, U10 TMP1826NG, U11 TMP1826NG, U12 TMP1826NG, U13 TMP1826NG, U14 TMP1826NG, U15 TMP1826NG, U16 TMP1826NG, U17 TMP1826NG, U18 TMP1826NG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

Commit message: All boards DRC/ERC clean
Routing:
- net +3.3V: track 184.6 -> 187.4 mm
- net GND: track 187.8 -> 190.0 mm
