File: Flow Shims/hardware/ts25/temp_sensors.kicad_sch (KiCad schematic)
At the start: 52 parts, among them J1 Conn_01x03, U10 TMP1826NG, U11 TMP1826NG, U12 TMP1826NG, U13 TMP1826NG, U14 TMP1826NG, U15 TMP1826NG, U16 TMP1826NG, U17 TMP1826NG, U18 TMP1826NG, U19 TMP1826NG, U2 TMP1826NG, U20 TMP1826NG, U21 TMP1826NG, U22 TMP1826NG, U23 TMP1826NG, U24 TMP1826NG, U25 TMP1826NG, U26 TMP1826NG, U3 TMP1826NG, U4 TMP1826NG, U5 TMP1826NG, U6 TMP1826NG, U7 TMP1826NG, U8 TMP1826NG, U9 TMP1826NG

Commit message: Single panel layout
Parts:
- removed J1: Conn_01x03, Connector_PinHeader_1.27mm:PinHeader_1x03_P1.27mm_Vertical, symbol Connector_Generic:Conn_01x03

Commit message: Building code for heater control PID loops
Parts:
- R1: value R_Small -> 2.2k
Changed lines of the file:
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@@
 			)
 		)
-		(property "Value" "R_Small"
+		(property "Value" "2.2k"
 			(at 226.06 69.8499 0)
 			(show_name no)
