File: Flow Shims/hardware/ts25/ts25.kicad_sch (KiCad schematic)
At the start: 24 parts, among them J2 Nano-Fit, U1 ADG5206, U27 ADG5206, U78 OPA196xDBV, U79 OPA196xDBV

Commit message: DRC clean, single heater
Parts:
- removed C55, C58: 100n, Capacitor_SMD:C_0603_1608Metric, symbol Device:C_Small
- removed U78, U79: OPA196xDBV, Package_TO_SOT_SMD:SOT-23-5, symbol Amplifier_Operational:OPA196xDBV
- added U28: OPA2196xDGK, Package_SO:VSSOP-8_3x3mm_P0.65mm, symbol Amplifier_Operational:OPA2196xDGK
- C26, C27, C28, C29, C56, C57: footprint Capacitor_SMD:C_0603_1608Metric -> Capacitor_SMD:C_0402_1005Metric
Connections:
- net +15V: now also U28.8 (V+)
- net -15V: now also U28.4 (V-)
- net VG: now also U28.7
- net VGIN: now also U28.3 (+)
- net at R4.2, R5.1: now also U28.5 (+)
- net at R2.1, R3.2: now also U28.2 (-)
- net at R2.2, R6.1, TP3.1: now also U28.1
- net at R6.2, R7.2: now also U28.6 (-)

Commit message: Building code for heater control PID loops
Other:
- note added: "Check Cap Voltage!"
Changed lines of the file:
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@@
 	(generator_version "10.0")
 	(paper "A4")
+	(text "Check Cap Voltage!"
+		(exclude_from_sim no)
+		(at 44.704 130.556 0)
+		(effects
+			(font
+				(size 1.27 1.27)
+			)
+		)
+	)
 	(junction
 		(at 147.32 41.91)
